Commit message: Added materials and IMU

File: urdf/materials.xacro (robot description, xacro)
@@ -1,4 +1,10 @@
 <?xml version="1.0" ?>
 <robot name="simple_robot_v2" xmlns:xacro="http://www.ros.org/wiki/xacro" >
+<material name="yellow">
+  <color rgba="0.800 0.500 0.000 1.000"/>
+</material>
+<material name="black">
+  <color rgba="0.000 0.000 0.000 1.000"/>
+</material>
 <material name="silver">
   <color rgba="0.700 0.700 0.700 1.000"/>

File: urdf/simple_robot_v2.xacro (robot description, xacro)
@@ -4,4 +4,6 @@
 <xacro:include filename="$(find simple_robot_v2_description)/urdf/simple_robot_v2.trans" />
 <xacro:include filename="$(find simple_robot_v2_description)/urdf/simple_robot_v2.gazebo" />
+<link name="dummy">
+</link>
 <link name="base_link">
   <inertial>
@@ -15,5 +17,5 @@
       <mesh filename="file://$(find simple_robot_v2_description)/meshes/base_link.stl" scale="0.001 0.001 0.001"/>
     </geometry>
-    <material name="silver"/>
+    <material name="yellow"/>
   </visual>
   <collision>
@@ -35,5 +37,5 @@
       <mesh filename="file://$(find simple_robot_v2_description)/meshes/left_wheel_1.stl" scale="0.001 0.001 0.001"/>
     </geometry>
-    <material name="silver"/>
+    <material name="black"/>
   </visual>
   <collision>
@@ -55,5 +57,5 @@
       <mesh filename="file://$(find simple_robot_v2_description)/meshes/right_wheel_1.stl" scale="0.001 0.001 0.001"/>
     </geometry>
-    <material name="silver"/>
+    <material name="black"/>
   </visual>
   <collision>
@@ -95,5 +97,5 @@
       <mesh filename="file://$(find simple_robot_v2_description)/meshes/lidar_cap_1.stl" scale="0.001 0.001 0.001"/>
     </geometry>
-    <material name="silver"/>
+    <material name="yellow"/>
   </visual>
   <collision>
@@ -104,4 +106,8 @@
   </collision>
 </link>
+<joint name="dummy_joint" type="fixed">
+  <parent link="dummy"/>
+  <child link="base_link"/>
+</joint>
 <joint name="Revolute 9" type="continuous">
   <origin xyz="-0.08 0.102 0.05" rpy="0 0 0"/>
